Commit message: reorganized

File: drone_description/urdf/camera.xacro (robot description, xacro)
@@ -5,5 +5,5 @@
     params="namespace parent_link robot_namespace camera_name image_topic_name camera_info_topic_name
       frame_rate horizontal_fov image_width image_height image_format min_distance
-      max_distance noise_mean noise_stddev enable_visual k1 k2 k3 p1 p2 cx cy *inertial *origin">
+      max_distance noise_mean noise_stddev enable_visual k1 k2 k3 p1 p2 cx cy *origin *visual *material">
     <joint name="${namespace}/${camera_name}_joint" type="fixed">
       <xacro:insert_block name="origin" />
@@ -12,15 +12,8 @@
     </joint>
     <link name="${namespace}/${camera_name}_link">
-      <xacro:insert_block name="inertial" />
-      <visual>
-        <origin xyz="0 0 0" rpy="0 0 0" />
-        <geometry>
-          <box size="0.008 0.02 0.012"/>
-        </geometry>
-        <xacro:material_orange/>
-      </visual>
+      <xacro:insert_block name="visual" />
     </link>
     <gazebo reference="${namespace}/${camera_name}_link">
-      <material>Gazebo/Orange</material>
+      <xacro:insert_block name="material" />
       <sensor type="camera" name="camera">
         <camera name="head">

File: drone_description/urdf/dji_m100_downward_camera.xacro (robot description, xacro)
@@ -28,11 +28,13 @@
     cx="0.5"
     cy="0.5">
-    <xacro:cylinder_inertial_with_origin
-      radius="0.01"
-      length="0.005"
-      mass="0.12">
+    <origin xyz="0 0 -0.1" rpy="0 ${pi/2} 0" />
+    <visual>
       <origin xyz="0 0 0" rpy="0 0 0" />
-    </xacro:cylinder_inertial_with_origin>
-    <origin xyz="0 0 -0.1" rpy="0 ${pi/2} 0" />
+      <geometry>
+        <box size="0.008 0.1 0.06"/>
+      </geometry>
+      <xacro:material_orange/>
+    </visual>
+    <material>Gazebo/Orange</material>
   </xacro:camera_macro>
   <xacro:if value="$(arg is_kinematic)">

File: drone_description/urdf/dji_m100_fpv.xacro (robot description, xacro)
@@ -28,11 +28,13 @@
     cx="0.5"
     cy="0.5">
-    <xacro:cylinder_inertial_with_origin
-      radius="0.01"
-      length="0.005"
-      mass="0.12">
+    <origin xyz="0 0 0.05" rpy="0 0 0" />
+    <visual>
       <origin xyz="0 0 0" rpy="0 0 0" />
-    </xacro:cylinder_inertial_with_origin>
-    <origin xyz="0 0 0.05" rpy="0 0 0" />
+      <geometry>
+        <box size="0.008 0.1 0.06"/>
+      </geometry>
+      <xacro:material_orange/>
+    </visual>
+    <material>Gazebo/Orange</material>
   </xacro:camera_macro>
   <xacro:if value="$(arg is_kinematic)">

File: drone_description/urdf/dji_m100_gimbal_camera.xacro (robot description, xacro)
@@ -36,11 +36,13 @@
     cx="0.5"
     cy="0.5">
-    <xacro:cylinder_inertial_with_origin
-      radius="0.01"
-      length="0.005"
-      mass="0.12">
+    <origin xyz="0.05 0 0" rpy="${pi/2} ${-pi/2} 0" />
+    <visual>
       <origin xyz="0 0 0" rpy="0 0 0" />
-    </xacro:cylinder_inertial_with_origin>
-    <origin xyz="0.05 0 0" rpy="${pi/2} ${-pi/2} 0" />
+      <geometry>
+        <box size="0.008 0.05 0.03"/>
+      </geometry>
+      <xacro:material_orange/>
+    </visual>
+    <material>Gazebo/Orange</material>
   </xacro:camera_macro>
   <xacro:if value="$(arg is_kinematic)">

File: drone_description/urdf/dji_m100_stereo_with_box.xacro (robot description, xacro)
@@ -30,11 +30,13 @@
     cx="0.5"
     cy="0.5">
-    <xacro:cylinder_inertial_with_origin
-      radius="0.01"
-      length="0.005"
-      mass="0.12">
+    <origin xyz="0 0.5 0" rpy="0 ${pi/2} 0" />
+    <visual>
       <origin xyz="0 0 0" rpy="0 0 0" />
-    </xacro:cylinder_inertial_with_origin>
-    <origin xyz="0 0.5 0" rpy="0 ${pi/2} 0" />
+      <geometry>
+        <box size="0.008 0.1 0.06"/>
+      </geometry>
+      <xacro:material_orange/>
+    </visual>
+    <material>Gazebo/Orange</material>
   </xacro:camera_macro>
   <xacro:camera_macro
@@ -62,11 +64,13 @@
     cx="0.5"
     cy="0.5">
-    <xacro:cylinder_inertial_with_origin
-      radius="0.01"
-      length="0.005"
-      mass="0.12">
+    <origin xyz="0 -0.5 0" rpy="0 ${pi/2} 0" />
+    <visual>
       <origin xyz="0 0 0" rpy="0 0 0" />
-    </xacro:cylinder_inertial_with_origin>
-    <origin xyz="0 -0.5 0" rpy="0 ${pi/2} 0" />
+      <geometry>
+        <box size="0.008 0.1 0.06"/>
+      </geometry>
+      <xacro:material_orange/>
+    </visual>
+    <material>Gazebo/Orange</material>
   </xacro:camera_macro>
   <link name="${namespace}/box_link">
