Commit message: tested on ubuntu18.04

File: uav_description/urdf/camera.xacro (robot description, xacro)
@@ -1,5 +1,5 @@
 <?xml version="1.0"?>
 <robot xmlns:xacro="http://ros.org/wiki/xacro">
-  <xacro:include filename="$(find drone_description)/urdf/common.xacro" />
+  <xacro:include filename="$(find uav_description)/urdf/common.xacro" />
   <xacro:macro name="camera_macro"
     params="namespace parent_link robot_namespace camera_name image_topic_name camera_info_topic_name

File: uav_description/urdf/dji_m100.xacro (robot description, xacro)
@@ -5,5 +5,5 @@
   <xacro:property name="rotor_velocity_slowdown_sim" value="10" />
   <xacro:property name="use_mesh_file" value="true" />
-  <xacro:property name="mesh_file" value="package://drone_description/meshes/dji_m100/dji_m100_flipped_rotorless.dae" />
+  <xacro:property name="mesh_file" value="package://uav_description/meshes/dji_m100/dji_m100_flipped_rotorless.dae" />
   <xacro:property name="mass" value="2.355" /> <!-- [kg] -->
   <xacro:property name="body_width" value="0.3" /> <!-- [m] -->
@@ -32,5 +32,5 @@
   </xacro:property>
   <!-- Included URDF Files -->
-  <xacro:include filename="$(find drone_description)/urdf/multirotor_base.xacro" />
+  <xacro:include filename="$(find uav_description)/urdf/multirotor_base.xacro" />
   <!-- Instantiate multirotor_base_macro once -->
   <xacro:multirotor_base_macro

File: uav_description/urdf/dji_m100_default.xacro (robot description, xacro)
@@ -2,5 +2,5 @@
 <robot name="dji_m100" xmlns:xacro="http://ros.org/wiki/xacro">
   <xacro:arg name="is_kinematic" default="true"/>
-  <xacro:include filename="$(find drone_description)/urdf/dji_m100.xacro" />
+  <xacro:include filename="$(find uav_description)/urdf/dji_m100.xacro" />
   <xacro:if value="$(arg is_kinematic)">
     <gazebo reference="${namespace}/base_link">

File: uav_description/urdf/dji_m100_downward_camera.xacro (robot description, xacro)
@@ -2,6 +2,6 @@
 <robot name="dji_m100" xmlns:xacro="http://ros.org/wiki/xacro">
   <xacro:arg name="is_kinematic" default="true"/>
-  <xacro:include filename="$(find drone_description)/urdf/dji_m100.xacro" />
-  <xacro:include filename="$(find drone_description)/urdf/camera.xacro" />
+  <xacro:include filename="$(find uav_description)/urdf/dji_m100.xacro" />
+  <xacro:include filename="$(find uav_description)/urdf/camera.xacro" />
   <xacro:camera_macro
     namespace="fixed_camera"

File: uav_description/urdf/dji_m100_fpv.xacro (robot description, xacro)
@@ -2,6 +2,6 @@
 <robot name="dji_m100" xmlns:xacro="http://ros.org/wiki/xacro">
   <xacro:arg name="is_kinematic" default="true"/>
-  <xacro:include filename="$(find drone_description)/urdf/dji_m100.xacro" />
-  <xacro:include filename="$(find drone_description)/urdf/camera.xacro" />
+  <xacro:include filename="$(find uav_description)/urdf/dji_m100.xacro" />
+  <xacro:include filename="$(find uav_description)/urdf/camera.xacro" />
   <xacro:camera_macro
     namespace="fixed_camera"

File: uav_description/urdf/dji_m100_gimbal_camera.xacro (robot description, xacro)
@@ -1,7 +1,7 @@
 <?xml version="1.0"?>
 <robot name="dji_m100" xmlns:xacro="http://ros.org/wiki/xacro">
-  <xacro:include filename="$(find drone_description)/urdf/dji_m100.xacro" />
-  <xacro:include filename="$(find drone_description)/urdf/gimbal.xacro" />
-  <xacro:include filename="$(find drone_description)/urdf/camera.xacro" />
+  <xacro:include filename="$(find uav_description)/urdf/dji_m100.xacro" />
+  <xacro:include filename="$(find uav_description)/urdf/gimbal.xacro" />
+  <xacro:include filename="$(find uav_description)/urdf/camera.xacro" />
   <!-- namespace indicate gazebo model namespace, see gazebo gui left panel -->
   <!-- robot_namespace is ros namespace -->

File: uav_description/urdf/dji_m100_stereo_with_box.xacro (robot description, xacro)
@@ -1,7 +1,7 @@
 <?xml version="1.0"?>
 <robot name="dji_m100" xmlns:xacro="http://ros.org/wiki/xacro">
-  <xacro:include filename="$(find drone_description)/urdf/dji_m100.xacro" />
-  <xacro:include filename="$(find drone_description)/urdf/gimbal.xacro" />
-  <xacro:include filename="$(find drone_description)/urdf/camera.xacro" />
+  <xacro:include filename="$(find uav_description)/urdf/dji_m100.xacro" />
+  <xacro:include filename="$(find uav_description)/urdf/gimbal.xacro" />
+  <xacro:include filename="$(find uav_description)/urdf/camera.xacro" />
   <!-- namespace indicate gazebo model namespace, see gazebo gui left panel -->
   <!-- robot_namespace is ros namespace -->

File: uav_description/urdf/gimbal.xacro (robot description, xacro)
@@ -1,5 +1,5 @@
 <?xml version="1.0"?>
 <robot xmlns:xacro="http://ros.org/wiki/xacro">
-  <xacro:include filename="$(find drone_description)/urdf/common.xacro" />
+  <xacro:include filename="$(find uav_description)/urdf/common.xacro" />
   <xacro:macro name="gazebo_ros_control_plugin_macro" params="namespace robot_namespace">
     <plugin name="${namespace}_gazebo_ros_control" filename="libgazebo_ros_control.so">

File: uav_description/urdf/multirotor_base.xacro (robot description, xacro)
@@ -73,5 +73,5 @@
           </xacro:if>
           <xacro:unless value="${use_own_mesh}">
-            <mesh filename="package://drone_description/meshes/propeller_${direction}.dae"
+            <mesh filename="package://uav_description/meshes/propeller_${direction}.dae"
               scale="${radius_rotor} ${radius_rotor} ${radius_rotor}" /> <!-- The propeller meshes have a radius of 1m -->
             <!-- <box size="${2*radius_rotor} 0.01 0.005"/> -->
